File: PJ6 - NE555 flow led/eagle/untitled.brd (EAGLE design)
At the start: 49 x 49 mm, 24 parts, among them IC2 CD4017, Q1 9013

Commit message: no message
Parts:
- added C4: 4.7uF, SparkFun-Capacitors:0603-CAP
- added D10, D11, D12, D13, D14, D15, D16, D17, D18, D19: (no value), SparkFun-LED:LED-1206
- added IC3: (no value), SparkFun-AnalogIC:SO08
- added IC4: 4017D, 40xx:SO16
- added Q2: 9013, SparkFun-DiscreteSemi:SOT23-3
- added R10, R11, R9: (no value), SparkFun-Resistors:0603-ARV
- added R6, R8: 470K, SparkFun-Resistors:0603-RES
- added R7: 10K, SparkFun-Resistors:0603-RES
- added TP1: TEST-POINT3, SparkFun-Passives:PAD.03X.03
- added U$2: (no value), r1:LOGO
- C1: value 100uF 5/6mm -> 100uF
- C2: value 4.7uF 5mm -> 4.7uF
- R1, R3: value 470K 1/4W -> 470K
- R2: value 10K 1/4W -> 10K
- moved BAT1 0.25 mm to (22.9, 37.1), flipped to the top, turned to 0 degrees
Connections:
- new net N$11: D12.A, IC4.4
- new net N$14: D13.A, IC4.7
- new net N$15: D14.A, IC4.10
- new net N$16: D15.A, IC4.1
- new net N$17: D16.A, IC4.5
- new net N$18: D17.A, IC4.6
- new net N$19: D18.A, IC4.9
- new net N$2: C1.1, Q1.2, Q2.1, R1.P$2, R6.2, S1.1, SJ1.1, TP1.P$1
- new net N$3: Q2.2, R7.2
- new net N$37: D19.A, IC4.11
- new net N$40: D10.C, R11.1
- new net N$41: D11.C, R11.2
- new net N$42: D12.C, R11.3
- new net N$43: D13.C, R11.4
- new net N$44: D14.C, R9.1
- new net N$45: D15.C, R9.2
- new net N$46: D16.C, R9.3
- new net N$47: D17.C, R9.4
- new net N$48: D18.C, R10.1
- new net N$49: D19.C, R10.2
- new net N$6: C4.1, IC3.2, IC3.6, IC3.7, R7.1, R8.2
- new net N$7: IC3.3, IC4.14
- new net N$8: D11.A, IC4.2
- net GND: now also C4.2, IC3.1, IC4.13, IC4.15, IC4.8, R10.7, R10.8, R11.5, R11.6, R11.7, R11.8, R6.1, R8.1, R9.5, R9.6, R9.7, R9.8
- net N$1: now also D10.A, IC4.3; no longer C1.1, Q1.2, R1.P$2, S1.1, SJ1.1
- net VCC: now also IC3.4, IC3.8, IC4.16, Q2.3
Routing:
- net N$1: track 36.1 -> 0.00 mm
- net VCC: vias 0 -> 1
Other:
- board text added: "NUPT SAST"
- board text added: "PJ6"
- board text added: "Rijn 2015"
- board text added: "mercury"
- board text added: "switch"
