File: PJ6 - NE555 flow led/eagle/untitled.sch (EAGLE design)
At the start: 24 parts, among them IC2 CD4017, Q1 9013

Commit message: no message
Parts:
- added C4: 4.7uF, SparkFun-Capacitors:4.7UF-6.3V-10%(0603)0603
- added D10, D11, D12, D13, D14, D15, D16, D17, D18, D19: (no value), SparkFun-LED:LED1206
- added IC3: (no value), SparkFun-AnalogIC:NE555D
- added IC4: 4017D, 40xx:4017D
- added Q2: 9013, SparkFun-DiscreteSemi:TRANSISTOR_NPNMMBT2222A
- added R10, R11, R9: (no value), SparkFun-Resistors:RESISTOR-ARRAY0603-ARV
- added R6, R8: 470K, SparkFun-Resistors:470OHM1/10W1%(0603)
- added R7: 10K, SparkFun-Resistors:470OHM1/10W1%(0603)
- added TP1: TEST-POINT3, SparkFun-Passives:TEST-POINT3
- C1: value 100uF 5/6mm -> 100uF
- C2: value 4.7uF 5mm -> 4.7uF
- R1, R3: value 470K 1/4W -> 470K
- R2: value 10K 1/4W -> 10K
Connections:
- new net N$11: D12.A, IC4A.Q2
- new net N$14: D13.A, IC4A.Q3
- new net N$15: D14.A, IC4A.Q4
- new net N$16: D15.A, IC4A.Q5
- new net N$17: D16.A, IC4A.Q6
- new net N$18: D17.A, IC4A.Q7
- new net N$19: D18.A, IC4A.Q8
- new net N$2: C1.+, Q1.B, Q2.B, R1.2, R6.2, S1.1, SJ1.1, TP1.1
- new net N$3: Q2.E, R7.2
- new net N$37: D19.A, IC4A.Q9
- new net N$40: D10.C, R11A.1
- new net N$41: D11.C, R11B.1
- new net N$42: D12.C, R11R.1
- new net N$43: D13.C, R11D.1
- new net N$44: D14.C, R9A.1
- new net N$45: D15.C, R9B.1
- new net N$46: D16.C, R9R.1
- new net N$47: D17.C, R9D.1
- new net N$48: D18.C, R10A.1
- new net N$49: D19.C, R10B.1
- new net N$6: C4.1, IC3.DIS, IC3.TRE, IC3.TRI, R7.1, R8.2
- new net N$7: IC3.OUT, IC4A.CLK
- new net N$8: D11.A, IC4A.Q1
- net GND: now also C4.2, IC3.GND, IC4A.ENA, IC4A.RES, IC4P.VSS, R10A.2, R10B.2, R11A.2, R11B.2, R11D.2, R11R.2, R6.1, R8.1, R9A.2, R9B.2, R9D.2, R9R.2
- net N$1: now also D10.A, IC4A.Q0; no longer C1.+, Q1.B, R1.2, S1.1, SJ1.1
- net VCC: now also IC3./RES, IC3.VCC+, IC4P.VDD, Q2.C
