File: PJ7 - SMDriver/eagle/pj7.sch (EAGLE design)
At the start: 41 parts, among them U2 PRTR5V0U2X, U3 CP210X_USB_UART, U4 STM32F103C8T

Commit message: no message
Parts:
- added STLINK: (no value), SparkFun-Connectors:M04LOCK
- added U6: MAX13488, SparkFun-DigitalIC:MAX13488
- renumbered U$1 to U5
Connections:
- net 3.3V: now also STLINK.1
- net GND: now also STLINK.2
- net SWCLK: now also STLINK.4
- net SWDIO: now also STLINK.3
Changed lines of the file:
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@@
 <part name="C16" library="SparkFun-Capacitors" deviceset="10NF/10000PF-50V-10%(0603)" device="" value="10nF"/>
 <part name="GND16" library="SparkFun-Aesthetics" deviceset="GND" device=""/>
-<part name="U$1" library="SparkFun-DigitalIC" deviceset="M93C46" device=""/>
+<part name="U5" library="SparkFun-DigitalIC" deviceset="M93C46" device=""/>
 <part name="R7" library="SparkFun-Resistors" deviceset="RESISTOR-ARRAY" device="0603-ARV"/>
 <part name="SJ4" library="SparkFun-Passives" deviceset="JUMPER-PTH-2-NO" device=""/>
+<part name="STLINK" library="SparkFun-Connectors" deviceset="M04" device="LOCK"/>
+<part name="U6" library="SparkFun-DigitalIC" deviceset="MAX13488" device=""/>
 </parts>
 <sheets>
@@
 <instance part="C16" gate="G$1" x="55.88" y="71.12"/>
 <instance part="GND16" gate="1" x="55.88" y="66.04"/>
-<instance part="U$1" gate="G$1" x="246.38" y="83.82"/>
+<instance part="U5" gate="G$1" x="246.38" y="83.82"/>
 <instance part="R7" gate="A" x="236.22" y="124.46"/>
 <instance part="R7" gate="B" x="236.22" y="119.38"/>
@@
 <instance part="R7" gate="D" x="236.22" y="109.22"/>
 <instance part="SJ4" gate="G$1" x="30.48" y="101.6"/>
+<instance part="STLINK" gate="G$1" x="137.16" y="104.14"/>
+<instance part="U6" gate="G$1" x="241.3" y="43.18"/>
 </instances>
 <busses>
@@
 <junction x="114.3" y="78.74"/>
 </segment>
+<segment>
+<pinref part="STLINK" gate="G$1" pin="1"/>
+<wire x1="147.32" y1="101.6" x2="142.24" y2="101.6" width="0.1524" layer="91"/>
+<label x="147.32" y="101.6" size="1.778" layer="95"/>
+</segment>
 </net>
 <net name="N$15" class="0">
@@
 <pinref part="GND16" gate="1" pin="GND"/>
 </segment>
+<segment>
+<pinref part="STLINK" gate="G$1" pin="2"/>
+<wire x1="147.32" y1="104.14" x2="142.24" y2="104.14" width="0.1524" layer="91"/>
+<label x="147.32" y="104.14" size="1.778" layer="95"/>
+</segment>
 </net>
 <net name="N$2" class="0">
@@
 <label x="203.2" y="50.8" size="1.778" layer="95"/>
 </segment>
+<segment>
+<pinref part="STLINK" gate="G$1" pin="4"/>
+<wire x1="142.24" y1="109.22" x2="147.32" y2="109.22" width="0.1524" layer="91"/>
+<label x="147.32" y="109.22" size="1.778" layer="95"/>
+</segment>
 </net>
 <net name="SWDIO" class="0">
@@
 <label x="203.2" y="48.26" size="1.778" layer="95"/>
 </segment>
-</net>
+<segment>
+<pinref part="STLINK" gate="G$1" pin="3"/>
+<wire x1="142.24" y1="106.68" x2="147.32" y2="106.68" width="0.1524" layer="91"/>
+<label x="147.32" y="106.68" size="1.778" layer="95"/>
+</segment>
+</net>

Commit message: 485
Parts:
- added C17: 0.1uF, SparkFun-Capacitors:0.1UF-25V-5%(0603)
- added R10, R11, R12, R13, R14, R8, R9: 10K, SparkFun-Resistors:10KOHM-1/10W-1%(0603)0603
- added R15, R16: (no value), SparkFun-Resistors:RESISTOR-ARRAY0603-ARV
- added SJ5, SJ6: JUMPER-PAD-3-2OF3_NC_BY_PASTE, SparkFun-Passives:JUMPER-PAD-3-2OF3_NC_BY_PASTE
- added U$1, U$2: TLP785, r1:TLP785
Connections:
- new net 485_A: R12.1, R14.2, U6.A
- new net 485_B: R12.2, R13.1, U6.B
- new net 485_RE: R16B.1
- new net 485_SHDN: R16R.1
- new net N$13: R15D.1, R8.1, U$1.4
- new net N$16: R9.1, U$2.1
- new net N$17: R15A.1, U$2.2
- new net N$19: R11.2, U$1.1
- new net N$22: R15R.1, R8.2
- new net N$23: R15B.1, R9.2
- new net N$24: R15A.2, R16A.2, U6.RO
- new net N$25: R15R.2, R16R.2, U6.SHDN
- new net N$26: R15D.2, R16D.2, U6.DI
- new net N$27: R15B.2, R16B.2, U6.RE
- new net N$28: R10.2, R16A.1, SJ6.2, U$2.4
- new net N$31: R16D.1, SJ5.2, U$1.2
- new net USART2_RX: SJ5.1, SJ6.3
- new net USART2_TX: SJ5.3, SJ6.1
- net 3.3V: now also C17.1, R10.1, R11.1, R14.1, U6.VCC
- net GND: now also C17.2, R13.2, U$1.3, U$2.3, U6.GND
Other:
- note added: "485"
- note added: "EEPROM"
- note added: "OLED"
- note added: "POWER"
- note added: "STM32"
- note added: "Serial"
- moved on the sheet: U6
