File: PJ7 - ServoDriver/eagle/pj7.brd (EAGLE design)
At the start: 80 x 80 mm, 136 parts, among them IC1 74HC595D, U2 PRTR5V0U2X, U3 CP210X_USB_UART, U4 STM32F103C8T, U5 M93C46, U6 MAX13488, U7 ADS1015

Commit message: no message
Parts:
- removed JP2: FTDI_DEVICE, SparkFun-Connectors:FTDI_DEVICE_SIDE
- removed R21, R41, R42: (no value), SparkFun-Resistors:0603-ARV
- added USART: (no value), SparkFun-Connectors:1X03_LOCK
- moved 433 56.9 mm to (60.5, 33.0), turned to 0 degrees
- moved S3 54.6 mm to (16.5, 26.9), turned to 0 degrees
- moved JP5 32.2 mm to (37.1, 4.83), turned to 0 degrees
- moved R20 26.6 mm to (44.5, 5.33), turned to 90 degrees
- moved SW1 25.1 mm to (73.2, 26.4)
- moved SJ3 24.2 mm to (48.3, 19.8), turned to 270 degrees
- moved C6 22.9 mm to (56.4, 25.1), turned to 270 degrees
- moved R40 22.6 mm to (39.6, 13.2), turned to 0 degrees
- moved R39 22.3 mm to (36.6, 13.2), turned to 180 degrees
- moved STLINK 21.9 mm to (30.5, 17.5), turned to 270 degrees
- moved SJ14 21.1 mm to (27.7, 26.9)
- moved D2 20.9 mm to (52.6, 22.6), turned to 0 degrees
- moved L1 20.7 mm to (56.4, 28.4), turned to 270 degrees
- moved R6 19.0 mm to (45.7, 19.8), turned to 270 degrees
- moved R18 18.5 mm to (78.5, 13.7), turned to 270 degrees
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Connections:
- removed net N$51: R42.1, SW1.9, U$9.4
- removed net N$52: R42.2, SW1.10, U$9.3
- removed net N$53: R42.3, SW1.11, U$9.2
- removed net N$54: R42.4, SW1.12, U$9.1
- net 3.3V: no longer R41.5, R41.6, R41.7, R41.8, R42.5, R42.6, R42.7, R42.8
- net 433_D0: now also SW1.9, U$9.4
- net 433_D1: now also SW1.10, U$9.3
- net 433_D2: now also SW1.11, U$9.2
- net 433_D3: now also SW1.12, U$9.1
- net 595_RCLK: now also U4.19; no longer U4.21
- net 595_SER: now also U4.18; no longer U4.22
- net 595_SRCLK: now also U4.21; no longer U4.19
- net 595_SRCLR: now also U4.22; no longer U4.18
- net GND: now also R20.3, USART.3; no longer JP2.P$6, R20.6
- net I2C1_SCL: now also R20.1; no longer R20.8
- net I2C1_SDA: now also R20.2; no longer R20.7
- net MP_A: now also U4.38
- net MP_S0: now also U4.39
- net MP_S1: now also U4.40
- net MP_S2: now also U4.41
- net N$55: no longer R41.1
- net N$56: no longer R41.2
- net N$57: no longer R41.3
- net N$58: no longer R41.4
- net OLED_CS: now also R20.6; no longer R20.3, R21.3, R21.6
- net OLED_SCL: now also R20.8; no longer R20.1, R21.1
- net OLED_SDA: now also R20.7; no longer R20.2, R21.2
- net SPI2_MOSI: no longer R21.7
- net SPI2_SCK: no longer R21.8
- net USART1_RX: now also USART.1; no longer JP2.P$2
- net USART1_TX: now also USART.2; no longer JP2.P$3
Routing:
- net 3.3V: track 0.00 -> 21.0 mm, vias 0 -> 2
- net N$12: track 0.00 -> 17.4 mm
- net D-: track 0.00 -> 15.2 mm, vias 0 -> 2
- net D+: track 0.00 -> 14.5 mm
- net N$5: track 0.00 -> 11.1 mm
- net GND: track 0.00 -> 3.76 mm
- net N$1: track 0.00 -> 3.04 mm

Commit message: no message
Parts:
- added U$1, U$2: (no value), r1:LOGO
- added U$10: (no value), logo:ESD_10.00
- moved M1 9.92 mm to (4.83, 42.9)
- moved SJ13 9.69 mm to (8.64, 48.0)
- moved SJ8 9.68 mm to (8.89, 38.4)
- moved M2 9.43 mm to (4.83, 33.3)
- moved SJ5 7.20 mm to (69.8, 56.6), turned to 270 degrees
- moved OS1 6.94 mm to (45.6, 25.3)
- moved D2 6.43 mm to (46.2, 22.6)
- moved SJ2 5.01 mm to (49.5, 25.2), turned to 270 degrees
- moved D11 4.66 mm to (11.2, 66.0), turned to 0 degrees
- moved R32 4.58 mm to (8.89, 63.8)
- moved U$6 4.31 mm to (65.9, 71.6)
- moved U$5 4.26 mm to (43.4, 71.6)
- moved R22 4.06 mm to (29.5, 49.8), turned to 270 degrees
- moved R23 4.06 mm to (31.5, 49.8), turned to 90 degrees
- moved R35 4.06 mm to (29.5, 53.8), turned to 90 degrees
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Connections:
- net N$8 renamed OURET
- net GND: now also R20.6, R7.1; no longer R20.3, R7.8
- net I2C1_SCL: now also R20.8; no longer R20.1
- net I2C1_SDA: now also R20.7; no longer R20.2
- net MP_A: no longer U4.33
- net N$63: now also R7.8; no longer R7.1
- net OLED_CS: now also R20.3; no longer R20.6
- net OLED_SCL: now also R20.1; no longer R20.8
- net OLED_SDA: now also R20.2; no longer R20.7
Routing:
- net 3.3V: track 21.0 -> 467.6 mm, vias 2 -> 14
- net VBUS: track 0.00 -> 196.9 mm, vias 0 -> 5
- net OLED_CS: track 0.00 -> 72.0 mm, vias 0 -> 3
- net TIM4_CH4: track 0.00 -> 66.9 mm, vias 0 -> 3
- net TIM4_CH3: track 0.00 -> 65.6 mm, vias 0 -> 3
- net OLED_RST: track 0.00 -> 63.7 mm, vias 0 -> 2
- net TIM1_CH4: track 0.00 -> 61.4 mm, vias 0 -> 1
- net OLED_DC: track 0.00 -> 58.3 mm, vias 0 -> 3
- net 485_SHDN: track 0.00 -> 49.9 mm
- net 485_RE: track 0.00 -> 48.9 mm
- net USART2_RX: track 0.00 -> 48.0 mm
- net TIM1_CH1: track 0.00 -> 46.4 mm, vias 0 -> 1
- net USART2_TX: track 0.00 -> 45.6 mm
- net USART1_RX: track 0.00 -> 37.9 mm, vias 0 -> 2
- net USART1_TX: track 0.00 -> 35.4 mm, vias 0 -> 2
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- added copper zone on layer 1, net GND
- added copper zone on layer 16, net GND
- added copper zone on layer 1, net V+
- added copper zone on layer 16, net V+
- added copper zone on layer 1, net V-
- added copper zone on layer 16, net V-
- added copper zone on layer 1, net VBUS
Other:
- outline, holes or cut-outs redrawn
- board text added: "DextaRobotics"
- board text added: "Oct 21, 2015"
- board text added: "PJ7"
- board text added: "STB REV A"
