File: PJ7 - ServoDriver/eagle/pj7.sch (EAGLE design)
At the start: 57 parts, among them U2 PRTR5V0U2X, U3 CP210X_USB_UART, U4 STM32F103C8T, U5 M93C46, U6 MAX13488

Commit message: no message
Parts:
- added C18, C22, C23: 0.1uF, SparkFun-Capacitors:0.1UF-25V-5%(0603)
- added C19, C20: 4.7uF, SparkFun-Capacitors:0.1UF-25V-5%(0603)
- added C21: 1uF, SparkFun-Capacitors:0.1UF-25V-5%(0603)
- added D4, D5, D6, D7: BAT54S, diode:BAT54S
- added JP3: (no value), SparkFun-Connectors:M03LOCK
- added L2: LBR2518T100K, eagle-ltspice:LL3225P
- added MBRM130LT3G: MBRA140, SparkFun-DiscreteSemi:MBRA140
- added OLED: (no value), SparkFun-Connectors:M07LOCK
- added R17: 330K, SparkFun-Resistors:10KOHM-1/10W-1%(0603)0603
- added R18, R19: 33K, SparkFun-Resistors:10KOHM-1/10W-1%(0603)0603
- added R20, R21: (no value), SparkFun-Resistors:RESISTOR-ARRAY0603-ARV
- added R22, R23: 10K, SparkFun-Resistors:10KOHM-1/10W-1%(0603)0603
- added SJ7, SJ8: JUMPER-PAD-3-2OF3_NC_BY_PASTE, SparkFun-Passives:JUMPER-PAD-3-2OF3_NC_BY_PASTE
- added U$3: LM2704, SparkFun-PowerIC:LM2704
- added U$4: 0.5_INCH_OLED, r1:0.5_INCH_OLED
- added U7: ADS1015, SparkFun-AnalogIC:ADS1118
- added V+, V-: (no value), SparkFun-Connectors:BANANA_CONN
Connections:
- new net 15V: C20.1, MBRM130LT3G.C, R17.2, U$4.VCC_C
- new net ADC_CS: U7.CS
- new net ANALOG_IN: D4.C1A2, U7.AIN2
- new net EEPROM_CS: U5.CS
- new net I1: D6.C1A2, U7.AIN0
- new net I2: D5.C1A2, U7.AIN1
- new net I2C1_SCL: R20A.2
- new net I2C1_SDA: R20B.2
- new net MOSI: R21B.2
- new net N$14: R17.1, R18.2, U$3.FB
- new net N$18: L2.2, MBRM130LT3G.A, U$3.SW
- new net N$20: C21.1, C22.1, U$4.VCC_R
- new net N$21: SJ7.2, U$4.IXS
- new net N$30: JP3.2, R22.2
- new net N$32: R19.1, U$4.IREF
- new net N$33: D7.C1A2, R22.1, R23.2, U7.AIN3
- new net N$36: JP3.3, SJ8.2
- new net OLED_CS: OLED.4, R20R.1, R21R.1, R21R.2, U$4.CSB
- new net OLED_DC: OLED.5, U$4.A0
- new net OLED_RST: OLED.3, U$4.RSTB
- new net OLED_SCL: OLED.7, R20A.1, R21A.1, U$4.D0/SCL
- new net OLED_SDA: OLED.6, R20B.1, R21B.1, U$4.D1/SI
- new net SPI1_MISO: U4MCU.PA6, U5.DOUT, U7.DOUT/DRDY
- new net SPI1_MOSI: U4MCU.PA7, U5.DIN, U7.DIN
- new net SPI1_SCK: U4MCU.PA5, U5.SK, U7.SCLK
- new net SPI2_CLK: R21A.2
- net 3.3V: now also C18.1, C19.1, C23.1, D4.C2, D5.C2, D6.C2, D7.C2, L2.1, OLED.2, SJ7.1, SJ8.1, U$3.SHDN, U$3.VIN, U$4.VDD, U5.VCC, U7.VDD
- net GND: now also C18.2, C19.2, C20.2, C21.2, C22.2, C23.2, D4.A1, D5.A1, D6.A1, D7.A1, JP3.1, OLED.1, R18.1, R19.2, R20R.2, R23.1, SJ7.3, U$3.GND, U$4.VSS, U5.GND, U7.VSS
- net VBUS: now also SJ8.3
Other:
- note added: "ADC"

Commit message: no message
Parts:
- added C25: 0.33uF, SparkFun-Capacitors:0.33UF-50V-10%(0805)
- added D10, D8, D9: BA340A, SparkFun-DiscreteSemi:B340A
- added D11: YELLOW, SparkFun-LED:LED-YELLOW1206
- added D12: RED, SparkFun-LED:LED-RED1206
- added JP4: (no value), SparkFun-Connectors:M02
- added R24, R25, R26, R27: 0.7K, SparkFun-Resistors:0OHM-1/10W-5%(0603)
- added R28, R29: 0, SparkFun-Resistors:0OHM-1/10W-5%(0603)
- added R30, R31: 0.001, SparkFun-Resistors:0.001OHM-3W-1%(2512)3W/1%
- added R32: 0.6K, SparkFun-Resistors:0.75OHM-1/4W-1%(0805)
- added S3: SWITCH-MOMENTARY-2SMD-12MM, SparkFun-Electromechanical:SWITCH-MOMENTARY-2SMD-12MM
- added SERVO1, SERVO2: (no value), SparkFun-Connectors:M03LOCK_LONGPADS
- added SJ10, SJ11, SJ12, SJ9: JUMPER-PAD-3-2OF3_NC_BY_PASTE, SparkFun-Passives:JUMPER-PAD-3-2OF3_NC_BY_PASTE
- added SW1: (no value), SparkFun-Electromechanical:SW_DIP-8-SMT-HALFSIZE
- added U$5, U$6: TLP785, SparkFun-DigitalIC:TLP785
- added U$7, U$8: INA282, SparkFun-PowerIC:INA282
- added U8: (no value), SparkFun-Electromechanical:ENCODER-QUADRATURE
- renumbered JP3 to M
Connections:
- removed net I1: D6.C1A2, U7.AIN0
- removed net I2: D5.C1A2, U7.AIN1
- new net N$29: R24.1, U$5.P$1
- new net N$34: R25.1, U$6.P$1
- new net N$35: R30.1, SERVO1.1, U$8.+IN
- new net N$37: R31.1, SERVO2.1, U$7.+IN
- new net N$38: R28.2, U$5.P$3
- new net N$39: R29.2, U$6.P$3
- new net N$40: SJ9.2, U$7.REF2
- new net N$41: SJ10.2, U$7.REF1
- new net N$42: SJ11.2, U$8.REF2
- new net N$43: SJ12.2, U$8.REF1
- new net N$44: D11.A, D12.C, R32.2
- new net PWM1: U$5.P$2
- new net PWM2: U$6.P$2
- new net S1: R26.1, SERVO1.3, U$5.P$4
- new net S2: R27.1, SERVO2.3, U$6.P$4
- new net SERVO1_OUTPUT: D6.C1A2, U$8.OUTPUT, U7.AIN0
- new net SERVO2_OUTPUT: D5.C1A2, U$7.OUTPUT, U7.AIN1
- new net V+: C25.1, D10.C, D8.C, D9.C, JP4.1, R26.2, R27.2, R32.1, SERVO1.2, SERVO2.2, V+.1
- new net V-: C25.2, D10.A, D11.C, D12.A, D8.A, D9.A, JP4.2, R28.1, R29.1, R30.2, R31.2, U$7.-IN, U$8.-IN, V-.1
- net 3.3V: now also R24.2, R25.2, SJ10.1, SJ11.3, SJ12.1, SJ9.3, U$7.V+, U$8.V+
- net GND: now also SJ10.3, SJ11.1, SJ12.3, SJ9.1, U$7.GND, U$8.GND
Other:
- note added: "433"
- note added: "Control"
- moved on the sheet: R7A, R7B, R7D, R7R, V-

Commit message: no message
Parts:
- removed M: (no value), SparkFun-Connectors:M03LOCK
- removed R10, R11, R8, R9: 10K, SparkFun-Resistors:10KOHM-1/10W-1%(0603)0603
- removed R15: (no value), SparkFun-Resistors:RESISTOR-ARRAY0603-ARV
- removed U$1, U$2: TLP785, r1:TLP785
- added 433: (no value), SparkFun-Connectors:M07LOCK
- added C24, C26, C27, C28: 0.1uF, SparkFun-Capacitors:0.1UF-25V-5%(0603)
- added D13, D14, D15: YELLOW, SparkFun-LED:LED-YELLOW1206
- added IC1: 74HC595D, 74xx-eu:74HC595D
- added JP5: (no value), SparkFun-Connectors:M03X2
- added JP6: (no value), SparkFun-Connectors:M02
- added M1, M2: (no value), SparkFun-Connectors:M03LOCK
- added R33, R34, R39, R40: 4.7K, SparkFun-Resistors:10KOHM-1/10W-1%(0603)0603
- added R35, R36, R43, R44, R45, R46: 10K, SparkFun-Resistors:10KOHM-1/10W-1%(0603)0603
- added R37, R38: 1K, SparkFun-Resistors:10KOHM-1/10W-1%(0603)0603
- added R41, R42: (no value), SparkFun-Resistors:RESISTOR-ARRAY0603-ARV
- added SJ13, SJ14: JUMPER-PAD-3-2OF3_NC_BY_PASTE, SparkFun-Passives:JUMPER-PAD-3-2OF3_NC_BY_PASTE
- added U$9: SN74CBT3251, SparkFun-DigitalIC:SN74CBT3251
Connections:
- removed net ANALOG_IN: D4.C1A2, U7.AIN2
- removed net MOSI: R21B.2
- removed net N$13: R15D.1, R8.1, U$1.4
- removed net PWM1: U$5.P$2
- removed net PWM2: U$6.P$2
- removed net SPI2_CLK: R21A.2
- new net 433_D0: 433.3
- new net 433_D1: 433.4
- new net 433_D2: 433.5
- new net 433_D3: 433.6
- new net 595_RCLK: IC1A.RCK, U4MCU.PB10
- new net 595_SER: IC1A.SER, U4MCU.PB11
- new net 595_SRCLK: IC1A.SCK, U4MCU.PB1
- new net 595_SRCLR: IC1A.SCL, U4MCU.PB0
- new net MP_A: U$9.A, U4MCU.PA12
- new net MP_S0: U$9.S0
- new net MP_S1: U$9.S1
- new net MP_S2: U$9.S2
- new net N$45: M1.3, SJ13.2
- new net N$46: D4.C1A2, R35.1, R36.2, U7.AIN2
- new net N$47: M1.2, R35.2
- new net N$48: R5.2, SJ14.2
- new net N$49: D5.C1A2, R43.1, R44.2, U7.AIN1
- new net N$50: D6.C1A2, R45.2, R46.1, U7.AIN0
- new net N$51: R42A.1, SW1.9, U$9.B1
- new net N$52: R42B.1, SW1.10, U$9.B2
- new net N$53: R42R.1, SW1.11, U$9.B3
- new net N$54: R42D.1, SW1.12, U$9.B4
- new net N$55: R41A.1, SW1.13, U$9.B5
- new net N$56: R41B.1, SW1.14, U$9.B6
- new net N$57: R41R.1, SW1.15, U$9.B7
- new net N$58: R41D.1, SW1.16, U$9.B8
- new net N$59: D13.C, R7B.2
- new net N$63: R7A.1, S3.2
- new net SPI2_MISO: U4MCU.PB14
- new net SPI2_MOSI: R21B.2, U4MCU.PB15
- new net SPI2_SCK: R21A.2, U4MCU.PB13
- new net SW: S3.1, U4MCU.PB12
- new net TIM1_CH1: U$5.P$2, U4MCU.PA8
- new net TIM1_CH4: U$6.P$2, U4MCU.PA11
- new net TIM4_CH3: R38.1, U4MCU.PB8, U8.B
- new net TIM4_CH4: R37.1, U4MCU.PB9, U8.A
- net 3.3V: now also C27.1, C28.1, D13.A, D14.A, D15.A, JP5.2, R33.2, R34.2, R37.2, R38.2, R39.2, R40.2, R41A.2, R41B.2, R41D.2, R41R.2, R42A.2, R42B.2, R42D.2, R42R.2, SJ13.1, SJ14.1; no longer R10.1, R11.1
- net 485_A: now also JP6.2
- net 485_B: now also JP6.1
- net 485_RE: now also U4MCU.PA1
- net 485_SHDN: now also U4MCU.PA0-WKUP
- net ADC_CS: now also IC1A.QD
- net EEPROM_CS: now also IC1A.QE
- net GND: now also 433.1, C24.2, C26.2, C27.2, C28.2, IC1A.G, IC1P.GND, JP5.1, JP5.3, JP5.5, M1.1, M2.1, R36.1, R44.1, R45.1, R7A.2, SJ14.3, SW1.1, SW1.2, SW1.3, SW1.4, SW1.5, SW1.6, SW1.7, SW1.8, U$9.GND, U$9.OE, U8.C; no longer M.1, R5.2, U$1.3, U$2.3
- net I2C1_SCL: now also JP5.4, R34.1, R39.1, U4MCU.PB6
- net I2C1_SDA: now also JP5.6, R33.1, R40.1, U4MCU.PB7
- net N$16: now also IC1A.QH, R7B.1; no longer R9.1, U$2.1
- net N$17: now also IC1A.QG, R7R.1; no longer R15A.1, U$2.2
- net N$19: now also IC1A.QF, R7D.1; no longer R11.2, U$1.1
- net N$22: now also D15.C, R7D.2; no longer R15R.1, R8.2
- net N$23: now also D14.C, R7R.2; no longer R15B.1, R9.2
- net N$24: no longer R15A.2
- net N$25: no longer R15R.2
- net N$26: no longer R15D.2
- net N$27: no longer R15B.2
- net N$28: no longer R10.2, U$2.4
- net N$30: now also M2.2; no longer M.2
- net N$31: no longer U$1.2
- net N$36: now also M2.3; no longer M.3
- net OLED_CS: now also IC1A.QB
- net OLED_DC: now also IC1A.QA
- net OLED_RST: now also IC1A.QC
- net SERVO1_OUTPUT: now also R46.2; no longer D6.C1A2, U7.AIN0
- net SERVO2_OUTPUT: now also R43.2; no longer D5.C1A2, U7.AIN1
- net USART2_RX: now also U4MCU.PA3
- net USART2_TX: now also U4MCU.PA2
- net VBUS: now also 433.2, C24.1, C26.1, IC1P.VCC, SJ13.3, U$9.VCC
Other:
- moved on the sheet: C18, C23, D4, D5, D6, D7, R22, R23, R7A, R7B, R7D, R7R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

Commit message: no message
Parts:
- removed JP2: FTDI_DEVICE, SparkFun-Connectors:FTDI_DEVICE
- removed R21, R41, R42: (no value), SparkFun-Resistors:RESISTOR-ARRAY0603-ARV
- added USART: (no value), SparkFun-Connectors:M03LOCK
Connections:
- removed net N$51: R42A.1, SW1.9, U$9.B1
- removed net N$52: R42B.1, SW1.10, U$9.B2
- removed net N$53: R42R.1, SW1.11, U$9.B3
- removed net N$54: R42D.1, SW1.12, U$9.B4
- net 3.3V: no longer R41A.2, R41B.2, R41D.2, R41R.2, R42A.2, R42B.2, R42D.2, R42R.2
- net 433_D0: now also SW1.9, U$9.B1
- net 433_D1: now also SW1.10, U$9.B2
- net 433_D2: now also SW1.11, U$9.B3
- net 433_D3: now also SW1.12, U$9.B4
- net 595_RCLK: now also U4MCU.PB1; no longer U4MCU.PB10
- net 595_SER: now also U4MCU.PB0; no longer U4MCU.PB11
- net 595_SRCLK: now also U4MCU.PB10; no longer U4MCU.PB1
- net 595_SRCLR: now also U4MCU.PB11; no longer U4MCU.PB0
- net GND: now also R20R.1, USART.3; no longer JP2.GND, R20R.2
- net I2C1_SCL: now also R20A.1; no longer R20A.2
- net I2C1_SDA: now also R20B.1; no longer R20B.2
- net MP_A: now also U4MCU.PA15
- net MP_S0: now also U4MCU.PB3
- net MP_S1: now also U4MCU.PB4
- net MP_S2: now also U4MCU.PB5
- net N$55: no longer R41A.1
- net N$56: no longer R41B.1
- net N$57: no longer R41R.1
- net N$58: no longer R41D.1
- net OLED_CS: now also R20R.2; no longer R20R.1, R21R.1, R21R.2
- net OLED_SCL: now also R20A.2; no longer R20A.1, R21A.1
- net OLED_SDA: now also R20B.2; no longer R20B.1, R21B.1
- net SPI2_MOSI: no longer R21B.2
- net SPI2_SCK: no longer R21A.2
- net USART1_RX: now also USART.1; no longer JP2.TXO
- net USART1_TX: now also USART.2; no longer JP2.RXI
Other:
- moved on the sheet: 433, R20A, R20B, R20D, R20R

Commit message: no message
Connections:
- net N$8 renamed OURET
- net GND: now also R20R.2, R7A.1; no longer R20R.1, R7A.2
- net I2C1_SCL: now also R20A.2; no longer R20A.1
- net I2C1_SDA: now also R20B.2; no longer R20B.1
- net MP_A: no longer U4MCU.PA12
- net N$63: now also R7A.2; no longer R7A.1
- net OLED_CS: now also R20R.1; no longer R20R.2
- net OLED_SCL: now also R20A.1; no longer R20A.2
- net OLED_SDA: now also R20B.1; no longer R20B.2
Other:
- moved on the sheet: R20A, R20B, R20D, R20R, R7A
Changed lines of the file:
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@@
 <instance part="GND16" gate="1" x="55.88" y="66.04"/>
 <instance part="U5" gate="G$1" x="266.7" y="81.28"/>
-<instance part="R7" gate="A" x="541.02" y="172.72"/>
+<instance part="R7" gate="A" x="541.02" y="172.72" rot="R180"/>
 <instance part="R7" gate="B" x="541.02" y="167.64"/>
 <instance part="R7" gate="R" x="541.02" y="162.56"/>
@@
 <instance part="SUPPLY20" gate="G$1" x="441.96" y="-15.24"/>
 <instance part="GND32" gate="1" x="444.5" y="-27.94"/>
-<instance part="R20" gate="A" x="515.62" y="96.52" rot="R180"/>
-<instance part="R20" gate="B" x="515.62" y="91.44" rot="R180"/>
-<instance part="R20" gate="R" x="515.62" y="86.36" rot="R180"/>
-<instance part="R20" gate="D" x="515.62" y="81.28" rot="R180"/>
+<instance part="R20" gate="A" x="515.62" y="96.52"/>
+<instance part="R20" gate="B" x="515.62" y="91.44"/>
+<instance part="R20" gate="R" x="515.62" y="86.36"/>
+<instance part="R20" gate="D" x="515.62" y="81.28"/>
 <instance part="GND33" gate="1" x="525.78" y="83.82"/>
 <instance part="D5" gate="G$1" x="454.66" y="5.08"/>
@@
 </segment>
 <segment>
-<pinref part="R20" gate="R" pin="1"/>
+<pinref part="R20" gate="R" pin="2"/>
 <wire x1="520.7" y1="86.36" x2="525.78" y2="86.36" width="0.1524" layer="91"/>
 <label x="525.78" y="86.36" size="1.778" layer="95"/>
@@
 <segment>
 <pinref part="GND54" gate="1" pin="GND"/>
-<pinref part="R7" gate="A" pin="2"/>
+<pinref part="R7" gate="A" pin="1"/>
 <wire x1="546.1" y1="172.72" x2="546.1" y2="182.88" width="0.1524" layer="91"/>
 <wire x1="546.1" y1="182.88" x2="571.5" y2="182.88" width="0.1524" layer="91"/>
@@
 </segment>
 </net>
-<net name="N$8" class="0">
+<net name="OURET" class="0">
 <segment>
 <pinref part="R5" gate="G$1" pin="1"/>
@@
 </segment>
 <segment>
-<pinref part="R20" gate="A" pin="2"/>
+<pinref part="R20" gate="A" pin="1"/>
 <wire x1="510.54" y1="96.52" x2="495.3" y2="96.52" width="0.1524" layer="91"/>
 <label x="495.3" y="96.52" size="1.778" layer="95"/>
@@
 </segment>
 <segment>
-<pinref part="R20" gate="B" pin="2"/>
+<pinref part="R20" gate="B" pin="1"/>
 <wire x1="495.3" y1="91.44" x2="510.54" y2="91.44" width="0.1524" layer="91"/>
 <label x="495.3" y="91.44" size="1.778" layer="95"/>
@@
 </segment>
 <segment>
-<pinref part="R20" gate="R" pin="2"/>
+<pinref part="R20" gate="R" pin="1"/>
 <wire x1="510.54" y1="86.36" x2="495.3" y2="86.36" width="0.1524" layer="91"/>
 <label x="495.3" y="86.36" size="1.778" layer="95"/>
@@
 <net name="I2C1_SCL" class="0">
 <segment>
-<pinref part="R20" gate="A" pin="1"/>
+<pinref part="R20" gate="A" pin="2"/>
 <wire x1="520.7" y1="96.52" x2="525.78" y2="96.52" width="0.1524" layer="91"/>
 <label x="525.78" y="96.52" size="1.778" layer="95"/>
@@
 <net name="I2C1_SDA" class="0">
 <segment>
-<pinref part="R20" gate="B" pin="1"/>
+<pinref part="R20" gate="B" pin="2"/>
 <wire x1="520.7" y1="91.44" x2="525.78" y2="91.44" width="0.1524" layer="91"/>
 <label x="525.78" y="91.44" size="1.778" layer="95"/>
@@
 </segment>
 <segment>
-<pinref part="U4" gate="MCU" pin="PA12"/>
-<wire x1="198.12" y1="45.72" x2="203.2" y2="45.72" width="0.1524" layer="91"/>
-<label x="203.2" y="45.72" size="1.778" layer="95"/>
-</segment>
-<segment>
 <pinref part="U4" gate="MCU" pin="PA15"/>
 <wire x1="203.2" y1="53.34" x2="198.12" y2="53.34" width="0.1524" layer="91"/>
@@
 <segment>
 <pinref part="S3" gate="G$1" pin="2"/>
-<pinref part="R7" gate="A" pin="1"/>
+<pinref part="R7" gate="A" pin="2"/>
 <wire x1="535.94" y1="172.72" x2="533.4" y2="172.72" width="0.1524" layer="91"/>
 <wire x1="533.4" y1="172.72" x2="533.4" y2="152.4" width="0.1524" layer="91"/>
