File: PJ9 - RELAY 51/eagle/pj9.brd (EAGLE design)
At the start: 50 x 50 mm, 28 parts, among them K1 G5LE

Commit message: no message
Parts:
- removed POWER2: (no value), SparkFun-Connectors:1X02_2.54_SCREWTERM
- added U$2: 2.1MMJACK, adafruit:PJ-102A
- added U$3: (no value), r1:LOGO
- moved D2 13.7 mm to (29.4, 9.32), turned to 90 degrees
- moved POWER3 8.98 mm to (26.7, 10.1)
- moved POWER1 1.19 mm to (5.16, 10.2)
- moved S1 0.95 mm to (25.2, 3.78)
Connections:
- removed net N$1: UART.1, UART_TP.7
- removed net N$6: UART.3, UART_TP.3
- removed net N$7: UART.4, UART_TP.1
- removed net N$9: SW1.11, SW1.12, UART_TP.6
- net 5V: now also UART.4, UART_TP.1
- net AGND: now also U$2.RING, U$2.RING_SW; no longer POWER2.P2
- net GND: now also UART.1, UART_TP.7
- net N$20: now also U$2.TIP; no longer POWER2.P1
- net N$3: now also SW1.11, SW1.12, UART_TP.6
- net N$8: now also UART.3, UART_TP.3
Routing:
- net N$20: track 9.63 -> 37.1 mm, vias 0 -> 1
- net AGND: track 0.00 -> 27.0 mm
- net N$3: track 4.64 -> 22.6 mm
- net N$9: track 12.1 -> 0.00 mm
- net N$8: track 15.1 -> 25.7 mm
- net 5V: track 104.3 -> 114.7 mm, vias 3 -> 4
- net N$6: track 4.90 -> 0.00 mm
- net N$1: track 4.90 -> 0.00 mm
- net N$7: track 4.64 -> 0.00 mm
- removed copper zone on layer 1, net AGND
- removed copper zone on layer 1, net N$20
Other:
- board text added: "PJ9"
- board text removed: "G"
