File: PJ9 - RELAY 51/eagle/pj9.sch (EAGLE design)
At the start: 28 parts, among them K1 G5LE

Commit message: no message
Parts:
- removed POWER2: (no value), SparkFun-Connectors:M022.54MM_SCREWTERM
- added U$2: 2.1MMJACK, adafruit:2.1MMJACK
Connections:
- removed net N$1: UART.1, UART_TP.7
- removed net N$6: UART.3, UART_TP.3
- removed net N$7: UART.4, UART_TP.1
- removed net N$9: SW1.11, SW1.12, UART_TP.6
- net 5V: now also UART.4, UART_TP.1
- net AGND: now also U$2.RING, U$2.RING_SW; no longer POWER2.2
- net GND: now also UART.1, UART_TP.7
- net N$20: now also U$2.TIP; no longer POWER2.1
- net N$3: now also SW1.11, SW1.12, UART_TP.6
- net N$8: now also UART.3, UART_TP.3
Changed lines of the file:
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@@
 <parts>
 <part name="POWER1" library="SparkFun-Connectors" deviceset="M02" device=""/>
-<part name="POWER2" library="SparkFun-Connectors" deviceset="M02" device="2.54MM_SCREWTERM"/>
 <part name="POWER3" library="SparkFun-Connectors" deviceset="M02" device="LOCK"/>
 <part name="D1" library="SparkFun-LED" deviceset="LED-YELLOW" device="1206" value="YELLOW"/>
@@
 <part name="GND8" library="SparkFun-Aesthetics" deviceset="GND" device=""/>
 <part name="JP3" library="SparkFun-Connectors" deviceset="M03X2" device=""/>
+<part name="U$2" library="adafruit" deviceset="2.1MMJACK" device=""/>
 </parts>
 <sheets>
@@
 <instances>
 <instance part="POWER1" gate="G$1" x="7.62" y="15.24"/>
-<instance part="POWER2" gate="G$1" x="7.62" y="27.94"/>
 <instance part="POWER3" gate="G$1" x="7.62" y="40.64"/>
 <instance part="D1" gate="G$1" x="35.56" y="68.58" rot="R270"/>
@@
 <instance part="GND8" gate="1" x="127" y="50.8"/>
 <instance part="JP3" gate="G$1" x="96.52" y="15.24" rot="R90"/>
+<instance part="U$2" gate="G$1" x="7.62" y="30.48"/>
 </instances>
 <busses>
@@
 <pinref part="POWER3" gate="G$1" pin="2"/>
 <wire x1="15.24" y1="43.18" x2="17.78" y2="43.18" width="0.1524" layer="91"/>
-<wire x1="17.78" y1="43.18" x2="17.78" y2="30.48" width="0.1524" layer="91"/>
-<pinref part="POWER2" gate="G$1" pin="2"/>
-<wire x1="17.78" y1="30.48" x2="15.24" y2="30.48" width="0.1524" layer="91"/>
-<wire x1="17.78" y1="30.48" x2="17.78" y2="17.78" width="0.1524" layer="91"/>
-<junction x="17.78" y="30.48"/>
+<wire x1="17.78" y1="43.18" x2="17.78" y2="27.94" width="0.1524" layer="91"/>
 <pinref part="POWER1" gate="G$1" pin="2"/>
+<wire x1="17.78" y1="27.94" x2="17.78" y2="17.78" width="0.1524" layer="91"/>
 <wire x1="17.78" y1="17.78" x2="15.24" y2="17.78" width="0.1524" layer="91"/>
 <wire x1="17.78" y1="43.18" x2="17.78" y2="53.34" width="0.1524" layer="91"/>
@@
 <wire x1="17.78" y1="53.34" x2="27.94" y2="53.34" width="0.1524" layer="91"/>
 <pinref part="D2" gate="G$1" pin="C"/>
+<label x="10.16" y="50.8" size="1.778" layer="95"/>
+<pinref part="U$2" gate="G$1" pin="RING"/>
+<wire x1="17.78" y1="27.94" x2="12.7" y2="27.94" width="0.1524" layer="91"/>
+<junction x="17.78" y="27.94"/>
+<pinref part="U$2" gate="G$1" pin="RING_SW"/>
+<wire x1="12.7" y1="30.48" x2="12.7" y2="27.94" width="0.1524" layer="91"/>
+<junction x="12.7" y="27.94"/>
 </segment>
 </net>
@@
 <wire x1="22.86" y1="91.44" x2="38.1" y2="91.44" width="0.1524" layer="91"/>
 <wire x1="38.1" y1="91.44" x2="38.1" y2="99.06" width="0.1524" layer="91"/>
+<pinref part="UART_TP" gate="G$1" pin="1"/>
+<pinref part="UART" gate="G$1" pin="4"/>
+<wire x1="0" y1="91.44" x2="7.62" y2="91.44" width="0.1524" layer="91"/>
+<wire x1="7.62" y1="91.44" x2="22.86" y2="91.44" width="0.1524" layer="91"/>
+<junction x="7.62" y="91.44"/>
+<junction x="22.86" y="91.44"/>
 </segment>
 <segment>
@@
 <pinref part="GND3" gate="1" pin="GND"/>
 <wire x1="22.86" y1="83.82" x2="25.4" y2="83.82" width="0.1524" layer="91"/>
+<pinref part="UART_TP" gate="G$1" pin="7"/>
+<pinref part="UART" gate="G$1" pin="1"/>
+<wire x1="0" y1="83.82" x2="7.62" y2="83.82" width="0.1524" layer="91"/>
+<wire x1="22.86" y1="83.82" x2="7.62" y2="83.82" width="0.1524" layer="91"/>
+<junction x="22.86" y="83.82"/>
+<junction x="7.62" y="83.82"/>
 </segment>
 <segment>
@@
 </segment>
 </net>
-<net name="N$1" class="0">
-<segment>
-<pinref part="UART_TP" gate="G$1" pin="7"/>
-<pinref part="UART" gate="G$1" pin="1"/>
-<wire x1="0" y1="83.82" x2="7.62" y2="83.82" width="0.1524" layer="91"/>
-</segment>
-</net>
 <net name="N$3" class="0">
 <segment>
@@
 <pinref part="UART" gate="G$1" pin="2"/>
 <wire x1="0" y1="86.36" x2="7.62" y2="86.36" width="0.1524" layer="91"/>
-</segment>
-</net>
-<net name="N$6" class="0">
-<segment>
-<pinref part="UART_TP" gate="G$1" pin="3"/>
-<pinref part="UART" gate="G$1" pin="3"/>
-<wire x1="0" y1="88.9" x2="7.62" y2="88.9" width="0.1524" layer="91"/>
-</segment>
-</net>
-<net name="N$7" class="0">
-<segment>
-<pinref part="UART_TP" gate="G$1" pin="1"/>
-<pinref part="UART" gate="G$1" pin="4"/>
-<wire x1="0" y1="91.44" x2="7.62" y2="91.44" width="0.1524" layer="91"/>
+<pinref part="UART_TP" gate="G$1" pin="6"/>
+<pinref part="SW1" gate="A" pin="11"/>
+<wire x1="22.86" y1="86.36" x2="40.64" y2="86.36" width="0.1524" layer="91"/>
+<wire x1="40.64" y1="86.36" x2="43.18" y2="86.36" width="0.1524" layer="91"/>
+<wire x1="40.64" y1="86.36" x2="40.64" y2="83.82" width="0.1524" layer="91"/>
+<junction x="40.64" y="86.36"/>
+<pinref part="SW1" gate="A" pin="12"/>
+<wire x1="40.64" y1="83.82" x2="43.18" y2="83.82" width="0.1524" layer="91"/>
+<wire x1="7.62" y1="86.36" x2="22.86" y2="86.36" width="0.1524" layer="91"/>
+<junction x="7.62" y="86.36"/>
+<junction x="22.86" y="86.36"/>
 </segment>
 </net>
@@
 <wire x1="40.64" y1="88.9" x2="43.18" y2="88.9" width="0.1524" layer="91"/>
 <junction x="40.64" y="88.9"/>
-</segment>
-</net>
-<net name="N$9" class="0">
-<segment>
-<pinref part="UART_TP" gate="G$1" pin="6"/>
-<pinref part="SW1" gate="A" pin="11"/>
-<wire x1="22.86" y1="86.36" x2="40.64" y2="86.36" width="0.1524" layer="91"/>
-<wire x1="40.64" y1="86.36" x2="43.18" y2="86.36" width="0.1524" layer="91"/>
-<wire x1="40.64" y1="86.36" x2="40.64" y2="83.82" width="0.1524" layer="91"/>
-<junction x="40.64" y="86.36"/>
-<pinref part="SW1" gate="A" pin="12"/>
-<wire x1="40.64" y1="83.82" x2="43.18" y2="83.82" width="0.1524" layer="91"/>
+<pinref part="UART_TP" gate="G$1" pin="3"/>
+<pinref part="UART" gate="G$1" pin="3"/>
+<wire x1="0" y1="88.9" x2="7.62" y2="88.9" width="0.1524" layer="91"/>
+<wire x1="22.86" y1="88.9" x2="7.62" y2="88.9" width="0.1524" layer="91"/>
+<junction x="22.86" y="88.9"/>
+<junction x="7.62" y="88.9"/>
 </segment>
 </net>
@@
 <pinref part="POWER1" gate="G$1" pin="1"/>
 <wire x1="15.24" y1="15.24" x2="20.32" y2="15.24" width="0.1524" layer="91"/>
-<wire x1="20.32" y1="15.24" x2="20.32" y2="27.94" width="0.1524" layer="91"/>
-<pinref part="POWER2" gate="G$1" pin="1"/>
-<wire x1="20.32" y1="27.94" x2="15.24" y2="27.94" width="0.1524" layer="91"/>
-<wire x1="20.32" y1="27.94" x2="20.32" y2="40.64" width="0.1524" layer="91"/>
-<junction x="20.32" y="27.94"/>
+<wire x1="20.32" y1="15.24" x2="20.32" y2="33.02" width="0.1524" layer="91"/>
 <pinref part="POWER3" gate="G$1" pin="1"/>
+<wire x1="20.32" y1="33.02" x2="20.32" y2="40.64" width="0.1524" layer="91"/>
 <wire x1="20.32" y1="40.64" x2="15.24" y2="40.64" width="0.1524" layer="91"/>
 <wire x1="20.32" y1="40.64" x2="20.32" y2="50.8" width="0.1524" layer="91"/>
@@
 <wire x1="20.32" y1="50.8" x2="43.18" y2="50.8" width="0.1524" layer="91"/>
 <pinref part="S1" gate="1" pin="P"/>
-</segment>
-</net>
+<pinref part="U$2" gate="G$1" pin="TIP"/>
+<wire x1="12.7" y1="33.02" x2="20.32" y2="33.02" width="0.1524" layer="91"/>
+<junction x="20.32" y="33.02"/>
+</segment>
+</net>
