File: PJ12 - Sensor/eagle/untitled.brd (EAGLE design)
At the start: 50 x 50 mm, 53 parts, among them U1 BMP180, Y1 8MHZ

Commit message: no message
Parts:
- removed SJ6: JUMPER-PAD-3-NC_BY_PASTE, SparkFun-Passives:PAD-JUMPER-3-NC_BY_PASTE_YES_SILK_FULL_BOX
- removed Y1: 8MHZ, SparkFun-FreqCtrl:RESONATOR-SMD
- added C15: 100nF, SparkFun-Capacitors:0603-CAP
- added C16, C19, C20: 33nF, SparkFun-Capacitors:0603-CAP
- added C17: 10nF, SparkFun-Capacitors:0603-CAP
- added C18: 1nF, SparkFun-Capacitors:0603-CAP
- added C21: 1.5pF, SparkFun-Capacitors:0603-CAP
- added C22: 1.0pF, SparkFun-Capacitors:0603-CAP
- added L2: 8.2nH, SparkFun-Passives:0603
- added L3: 3.9nH, SparkFun-Passives:0603
- added L4: 2.7nH, SparkFun-Passives:0603
- added OS1: OSC-OE-IQXO-793, IQD-Frequency-Products:2.5X2-4-PAD
- added R11: 22K, SparkFun-Resistors:0603
- added U$12, U$13: JUMPER_PAD-3-1&2_NC_BY_PASTE, SparkFun-Passives:PAD-HUMPER-3-1&2_NC_BY_PASTE_YES_SILK_FULL_BOX
- added U$14: ANTENNA2SMD2, SparkFun-RF:ANTENNA-CHIP3
Connections:
- removed net DVDD: U$5.19
- removed net VDD_PA: U$5.11
- removed net VSS: U$5.0, U$5.14, U$5.17, U$5.20, U$5.8
- new net CLK_16M: OS1.3, U$5.10, U$7.2
- new net N$14: L2.2, L4.1, U$5.12
- new net N$16: C15.2, OS1.2, U$12.3
- new net N$28: OS1.1, U$12.2
- new net N$29: C16.1, U$5.19
- new net N$30: R11.1, U$5.16
- new net N$32: C21.1, L3.2
- new net N$33: C21.2, C22.1, U$14.FEED
- net GND: now also C16.2, C17.2, C18.2, C19.2, C20.2, C22.2, R11.2, U$13.1, U$5.0, U$5.14, U$5.17, U$5.20, U$5.8; no longer SJ6.3, Y1.2
- net MESH: no longer U$5.15, U$5.18, U$5.7
- net N$11: now also L2.1, L3.1, U$5.13; no longer U$7.2, Y1.1
- net N$24: now also C19.1, C20.1, L4.2, U$5.11; no longer U$7.3, Y1.3
- net N$25: now also U$13.2; no longer SJ6.2
- net NRF_CE: now also U$5.1
- net NRF_CSN: now also U$5.2
- net NRF_IRQ: now also U$5.6
- net RST: now also JP3.7; no longer JP3.3
- net SPI1_MISO: now also U$5.5
- net SPI1_MOSI: now also U$5.4
- net SPI1_SCK: now also U$5.3
- net SWCLK: now also JP3.5; no longer JP3.7
- net SWDIO: now also JP3.3; no longer JP3.5
- net VDD: now also C15.1, C17.1, C18.1, OS1.4, U$12.1, U$13.3, U$5.15, U$5.18, U$5.7; no longer SJ6.1
