File: PJ12 - Sensor/eagle/untitled.sch (EAGLE design)
At the start: 51 parts, among them U1 BMP180, Y1 8MHZ

Commit message: no message
Parts:
- removed SJ6: JUMPER-PAD-3-NC_BY_PASTE, SparkFun-Passives:JUMPER-PAD-3-NC_BY_PASTE
- removed Y1: 8MHZ, SparkFun-FreqCtrl:RESONATOR8MHZ
- added C15: 100nF, SparkFun-Capacitors:0.1UF-25V-5%(0603)
- added C16, C19, C20: 33nF, SparkFun-Capacitors:0.1UF-25V-5%(0603)
- added C17: 10nF, SparkFun-Capacitors:0.1UF-25V-5%(0603)
- added C18: 1nF, SparkFun-Capacitors:0.1UF-25V-5%(0603)
- added C21: 1.5pF, SparkFun-Capacitors:0.1UF-25V-5%(0603)
- added C22: 1.0pF, SparkFun-Capacitors:0.1UF-25V-5%(0603)
- added L2: 8.2nH, SparkFun-Passives:INDUCTOR0603
- added L3: 3.9nH, SparkFun-Passives:INDUCTOR0603
- added L4: 2.7nH, SparkFun-Passives:INDUCTOR0603
- added OS1: OSC-OE-IQXO-793, IQD-Frequency-Products:OSC-OE-IQXO-793
- added R11: 22K, SparkFun-Resistors:1.5KOHM-1/10W-1%(0603)
- added U$12, U$13: JUMPER_PAD-3-1&2_NC_BY_PASTE, SparkFun-Passives:JUMPER_PAD-3-1&2_NC_BY_PASTE
- added U$14: ANTENNA2SMD2, SparkFun-RF:ANTENNA2SMD2
Connections:
- new net CLK_16M: OS1.OUT, U$5.XC1, U$7.PF0-OSC_IN
- new net N$14: L2.2, L4.1, U$5.ANT1
- new net N$16: C15.2, OS1.VSS, U$12.3
- new net N$28: OS1.CON, U$12.2
- new net N$29: C16.1, U$5.DVDD
- new net N$30: R11.1, U$5.IREF
- new net N$32: C21.1, L3.2
- new net N$33: C21.2, C22.1, U$14.SIGNAL
- net GND: now also C16.2, C17.2, C18.2, C19.2, C20.2, C22.2, R11.2, U$13.1, U$5.VSS@0, U$5.VSS@14, U$5.VSS@17, U$5.VSS@20, U$5.VSS@8; no longer SJ6.3, Y1.2
- net N$11: now also L2.1, L3.1, U$5.ANT2; no longer U$7.PF0-OSC_IN, Y1.1
- net N$24: now also C19.1, C20.1, L4.2, U$5.VDD_PA; no longer U$7.PF1-OSC_OUT, Y1.3
- net N$25: now also U$13.2; no longer SJ6.2
- net NRF_CE: now also U$5.CE
- net NRF_CSN: now also U$5.CSN
- net NRF_IRQ: now also U$5.IRQ
- net RST: now also JP3.7; no longer JP3.3
- net SPI1_MISO: now also U$5.MISO
- net SPI1_MOSI: now also U$5.MOSI
- net SPI1_SCK: now also U$5.SCK
- net SWCLK: now also JP3.5; no longer JP3.7
- net SWDIO: now also JP3.3; no longer JP3.5
- net VDD: now also C15.1, C17.1, C18.1, OS1.VDD, U$12.1, U$13.3, U$5.VDD@15, U$5.VDD@18, U$5.VDD@7; no longer SJ6.1
Other:
- moved on the sheet: U$5
