File: PJ12 - Sensor/eagle/pj12.sch (EAGLE design)
At the start: 65 parts, among them U1 BMP180

Commit message: update pj13 & pj15
Parts:
- removed SJ4: JUMPER-PAD-3-NC_BY_PASTE, SparkFun-Passives:JUMPER-PAD-3-NC_BY_PASTE
- removed U$11: TPS61291, r1:TPS61291
- removed U$6: NRF24L01_MODULE_SMD, User-Submitted:NRF24L01_MODULE_SMD
- added U7: BMP180, SparkFun-Sensors:BMP180
- U1: value BMP180 -> TPS61291; device SparkFun-Sensors:BMP180 -> r1:TPS61291
- renumbered OS1 to U5, U$2 to U2, U$3 to U3, U$4 to U6, U$5 to U9, U$7 to U4, U$8 to U8
Connections:
- removed net MESH: C1.+, C10.1, C11.1, C12.1, C7.1, C8.1, C9.1, R10.2, R8.1, R9.1, SJ2.1, SJ3.2, SJ5.3, U$6.VCC, U1.VDD, U1.VDDIO, U8.VCC
- removed net N$26: JP3.8, SJ4.2
- net GND: now also JP3.8, U7.GND; no longer SJ4.3, U$11.GND, U$6.GND
- net I2C1_SCL: now also U7.SCL; no longer U1.SCL
- net I2C1_SDA: now also U7.SDA; no longer U1.SDA
- net N$3: now also U1.SW; no longer U$11.SW
- net N$4: now also U1.VOUT; no longer U$11.VOUT
- net N$5: now also U1.EN/BYP; no longer U$11.EN/BYP
- net N$6: now also U1.VSEL; no longer U$11.VSEL
- net NRF_CE: no longer U$6.CE
- net NRF_CSN: no longer U$6.CSN
- net NRF_IRQ: no longer U$6.IRQ
- net PB1: no longer SJ4.1
- net SPI1_MISO: no longer U$6.MISO
- net SPI1_MOSI: no longer U$6.MOSI
- net SPI1_SCK: no longer U$6.SCK
- net VDD: now also C1.+, C10.1, C11.1, C12.1, C7.1, C8.1, C9.1, R10.2, R8.1, R9.1, SJ2.1, SJ3.2, SJ5.3, U7.VDD, U7.VDDIO, U8.VCC
- net V_BATT: now also U1.VIN; no longer U$11.VIN
