File: MB2 - STM32F407VET6/eagle/mb2.sch (EAGLE design)
At the start: 57 parts, among them Q1 FC-12M, U1 MIC5219 3.3V

Commit message: update pj13 & pj15
Parts:
- removed G1: CH291-1220LF, battery:CH291-1220LF
- removed JP1: (no value), SparkFun-Connectors:M03LOCK
- added C35: 0.1uF, SparkFun-Capacitors:0.1UF-25V-5%(0603)
- added GPIO1, GPIO2, GPIO3: (no value), SparkFun-Connectors:M13X22X13
- added POWER: (no value), SparkFun-Connectors:M03X22X3_SILK_MALE_PTH
- added R10, R11: (no value), SparkFun-Resistors:RESISTOR-ARRAY0603-ARV
- added U$5: SPI_FLASH-X25XXSMD, SparkFun-DigitalIC:SPI_FLASH-X25XXSMD
- added U2: USD-SOCKETNEW, SparkFun-Connectors:USD-SOCKETNEW
- added VBAT: JUMPER-PAD-2-NC_BY_TRACE, SparkFun-Passives:JUMPER-PAD-2-NC_BY_TRACE
Connections:
- removed net BAT: G1.+, JP1.3
- removed net BOOT0: INTERFACE.4
- removed net RX: INTERFACE.9
- removed net TX: INTERFACE.10
- new net PA0: U$1.PA0/WKUP
- new net PA1: U$1.PA1
- new net PA10: INTERFACE.1, U$1.PA10
- new net PA11: U$1.PA11
- new net PA12: U$1.PA12
- new net PA15: U$1.PA15
- new net PA2: U$1.PA2
- new net PA3: U$1.PA3
- new net PA4: U$1.PA4, U$5.CS
- new net PA5: U$1.PA5, U$5.SCK
- new net PA6: U$1.PA6, U$5.MISO
- new net PA7: U$1.PA7, U$5.MOSI
- new net PA8: U$1.PA8
- new net PA9: INTERFACE.2, U$1.PA9
- new net PB0: U$1.PB0
- new net PB1: U$1.PB1
- new net PB10: U$1.PB10
- new net PB11: U$1.PB11
- new net PB12: U$1.PB12
- new net PB13: U$1.PB13
- new net PB14: U$1.PB14
- new net PB15: U$1.PB15
- new net PB3: U$1.PB3
- new net PB4: U$1.PB4
- new net PB5: U$1.PB5
- new net PB6: U$1.PB6
- new net PB7: U$1.PB7
- new net PB8: U$1.PB8
- new net PB9: U$1.PB9
- new net PC0: U$1.PC0
- new net PC1: U$1.PC1
- new net PC10: R10D.1, U$1.PC10, U2.NC
- new net PC11: R10R.1, U$1.PC11, U2.CS
- new net PC12: R10A.1, U$1.PC12, U2.SCK
- new net PC13: U$1.PC13
- new net PC2: U$1.PC2
- new net PC3: U$1.PC3
- new net PC4: U$1.PC4
- new net PC5: U$1.PC5
- new net PC6: U$1.PC6
- new net PC7: U$1.PC7
- new net PC8: R11D.1, U$1.PC8, U2.DO
- new net PC9: R11R.1, U$1.PC9, U2.RSV
- new net PD0: U$1.PD0
- new net PD1: U$1.PD1
- new net PD10: U$1.PD10
- new net PD11: U$1.PD11
- new net PD12: U$1.PD12
- new net PD13: U$1.PD13
- new net PD14: U$1.PD14
- new net PD15: U$1.PD15
- new net PD2: R10B.1, U$1.PD2, U2.DI
- new net PD3: U$1.PD3
- new net PD4: U$1.PD4
- new net PD5: U$1.PD5
- new net PD6: U$1.PD6
- new net PD7: U$1.PD7
- new net PD8: U$1.PD8
- new net PD9: U$1.PD9
- new net PE0: U$1.PE0
- new net PE1: U$1.PE1
- new net PE10: U$1.PE10
- new net PE11: U$1.PE11
- new net PE12: U$1.PE12
- new net PE13: U$1.PE13
- new net PE14: U$1.PE14
- new net PE15: U$1.PE15
- new net PE2: U$1.PE2
- new net PE3: U$1.PE3
- new net PE4: U$1.PE4
- new net PE5: U$1.PE5
- new net PE6: U$1.PE6
- new net PE7: U$1.PE7
- new net PE8: U$1.PE8
- new net PE9: U$1.PE9
- net 3.3V: now also C35.2, INTERFACE.10, POWER.3, POWER.5, R10A.2, R10B.2, R10D.2, R10R.2, R11A.2, R11B.2, R11D.2, R11R.2, U$5.HOLD, U$5.VCC, U$5.WP, U2.VCC, VBAT.2; no longer INTERFACE.2, JP1.1
- net 5V: now also INTERFACE.9, POWER.1; no longer INTERFACE.1
- net GND: now also C35.1, INTERFACE.4, POWER.2, POWER.4, POWER.6, U$5.GND, U2.CD1, U2.CD2, U2.GND, U2.SHIELD@1, U2.SHIELD@3; no longer G1.-
- net N$5: now also VBAT.1; no longer JP1.2
